File: smeza_pcb/smeza_pcb.kicad_sch (KiCad schematic)
At the start: 50 parts, among them J1 SS-90000-002, J2 SS-90000-002, J3 Conn_01x03, J4 Conn_01x04, J5 Conn_01x03, J6 Conn_01x03, J7 Conn_01x03, J8 Conn_01x03, J9 Conn_02x03_Odd_Even, SW1 SW_DIP_x04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

Commit message: Changed library paths from absolute paths to relative paths. Attempted to fix issue referencing old versions of the schematic.
Parts:
- B1: footprint SOIC127P600X170-9N -> Footprints:SOIC127P600X170-9N
- H1: footprint H-bridge:SOIC100P600X175-10N -> Footprints:SOIC100P600X175-10N
- J1: footprint SS-90000-002:SS90000002 -> Footprints:SS90000002
- T1: footprint ADM4852ARZ:ADM4852ARZ -> Footprints:ADM4852ARZ

Commit message: Corrected Footprints in Schematic. Reorganized passives supporting the buck converter. Rerouted 50V passthough, D+/- passthrough.
Connections:
- net BuckConverterVCC: now reaches B1.2 (VCC), C6.2
Changed lines of the file:
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@@
+    (effects (font (size 1.27 1.27)) (justify left bottom))
+  )
+  (label "BuckConverterVCC" (at 124.46 190.5 0) (fields_autoplaced)
     (effects (font (size 1.27 1.27)) (justify left bottom))
   )

Commit message: Reorganized all components and rerouted. Added capacitors to H-Bridge. Added Capacitors to dip switches. Updated DIP switch footprint. Fixed DRC and ERC errors.
Parts:
- added C10, C11, C9: 1nF, Capacitor_SMD:C_1206_3216Metric, symbol Device:C
- added C8: 10uF, Capacitor_SMD:C_1206_3216Metric, symbol Device:C
- added Y1: CSTNE16M0V530000R0, Footprints:OSC_CSTNE16M0V530000R0, symbol CSTNE16M0V530000R0:CSTNE16M0V530000R0
- H1: symbol H_bridge:H_Bridge -> A3909GLNTR-T:A3909GLNTR-T; Arrow Part Number (none) -> A3909GLNTR-T; Arrow Price/Stock (none) -> https://www.arrow.com/en/products/a3909glntr-t/allegro-micr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; Height (none) -> 1.75; Manufacturer_Name (none) -> Allegro Microsystems; Manufacturer_Part_Number (none) -> A3909GLNTR-T; Mouser Part Number (none) -> 250-A3909GLNTR-T; Mouser Price/Stock (none) -> https://www.mouser.co.uk/ProductDetail/Allegro-MicroSystems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
- J1, U1: now not fitted
- J2: footprint SS-90000-002:SS90000002 -> Footprints:SS90000002; now not fitted
- J9: footprint Connector_PinHeader_2.00mm:PinHeader_2x03_P2.00mm_Vertical -> Connector_PinHeader_2.54mm:PinHeader_2x03_P2.54mm_Vertical
- R4: value DNP -> 120; now not fitted
- SW1, SW2: footprint Button_Switch_SMD:SW_DIP_SPSTx04_Slide_6.7x11.72mm_W8.61mm_P2.54mm_LowProfile -> Button_Switch_THT:SW_DIP_SPSTx04_Slide_9.78x12.34mm_W7.62mm_P2.54mm
- SW3: footprint Button_Switch_SMD:SW_DIP_SPSTx01_Slide_6.7x4.1mm_W8.61mm_P2.54mm_LowProfile -> Button_Switch_THT:SW_DIP_SPSTx01_Slide_9.78x4.72mm_W7.62mm_P2.54mm
Connections:
- net +5V: now also C8.1
- net DIP9: now also C11.1
- net DIPS14: now also C9.1
- net DIPS58: now also C10.1
- net GND: now also C10.2, C11.2, C8.2, C9.2, Y1.2
- net at U2.7 (XTAL1/PB6): now also Y1.1
- net at U2.8 (XTAL2/PB7): now also Y1.3
- no-connect marks 0 -> 7
Other:
- note added: "ICSP Header"
- moved on the sheet: D1, J4, R22

Commit message: Separated MOSI and M2 Bkwd pins
Connections:
- net M2 Bkwd Signal: now reaches U2.12 (PB0)
- net M2 Bkwd Signal: now also H1.4 (IN3)
- net M2 Bkwd Signal (MOSI) renamed MOSI
- net MOSI: no longer H1.4 (IN3)
- no-connect marks 7 -> 6
Changed lines of the file:
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@@
   (no_connect (at 311.15 116.84))
   (no_connect (at 311.15 121.92))
-  (no_connect (at 311.15 63.5))
   (no_connect (at 311.15 91.44))
   (wire (pts (xy 411.48 166.37) (xy 424.815 166.37))
@@
     (stroke (width 0) (type default))
   )
+  (wire (pts (xy 311.15 63.5) (xy 402.59 63.5))
+    (stroke (width 0) (type default))
+  )
   (wire (pts (xy 41.91 201.93) (xy 41.91 204.47))
     (stroke (width 0) (type default))
@@
     (stroke (width 0) (type default))
   )
-  (wire (pts (xy 402.59 66.04) (xy 402.59 83.82))
+  (wire (pts (xy 402.59 63.5) (xy 402.59 83.82))
     (stroke (width 0) (type default))
   )
@@
     (stroke (width 0) (type default))
   )
-  (wire (pts (xy 311.15 66.04) (xy 402.59 66.04))
-    (stroke (width 0) (type default))
-  )
   (wire (pts (xy 127 198.12) (xy 127 193.04))
     (stroke (width 0) (type default))
@@
   )
   (wire (pts (xy 92.71 102.87) (xy 102.87 102.87))
+    (stroke (width 0) (type default))
+  )
+  (wire (pts (xy 311.15 66.04) (xy 327.66 66.04))
     (stroke (width 0) (type default))
   )
@@
     (effects (font (size 1.27 1.27)) (justify left bottom))
   )
+  (label "MOSI" (at 313.055 66.04 0) (fields_autoplaced)
+    (effects (font (size 1.27 1.27)) (justify left bottom))
+  )
   (label "+5V" (at 386.715 233.68 0) (fields_autoplaced)
     (effects (font (size 1.27 1.27)) (justify left bottom))
@@
     (effects (font (size 1.27 1.27)) (justify left bottom))
   )
-  (label "M2 Bkwd Signal (MOSI)" (at 443.865 231.14 0) (fields_autoplaced)
+  (label "MOSI" (at 443.865 231.14 0) (fields_autoplaced)
     (effects (font (size 1.27 1.27)) (justify left bottom))
   )
@@
     (effects (font (size 1.27 1.27)) (justify left bottom))
   )
-  (label "M2 Bkwd Signal (MOSI)" (at 313.055 66.04 0) (fields_autoplaced)
-    (effects (font (size 1.27 1.27)) (justify left bottom))
-  )
+  (label "M2 Bkwd Signal" (at 313.055 63.5 0) (fields_autoplaced)
+    (effects (font (size 1.27 1.27)) (justify left bottom))
+  )

Commit message: Replaced most extended parts. Swapped out many 1206 resistors for 0805 resistors. Swapped out C1. Swapped out LED. Made all headers DNP. Rerouted to reflect the new footprints.
Parts:
- B1, J3, J4, J5, J6, J7, J8, J9, SW1, SW2, SW3: now not fitted
- C1: footprint Capacitor_SMD:C_1206_3216Metric -> Capacitor_SMD:C_0603_1608Metric
- D1: footprint LED_SMD:LED_1206_3216Metric -> LED_SMD:LED_0603_1608Metric
- R1, R10, R11, R12, R13, R14, R15, R16, R17, R18, R19, R2, R20, R21, R22, R4, R5, R6, R7, R8, R9: footprint Resistor_SMD:R_1206_3216Metric -> Resistor_SMD:R_0805_2012Metric
Changed lines of the file:
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@@
       (effects (font (size 1.27 1.27)))
     )
-    (property "Footprint" "Resistor_SMD:R_1206_3216Metric" (at 217.17 342.138 90)
+    (property "Footprint" "Resistor_SMD:R_0805_2012Metric" (at 217.17 342.138 90)
       (effects (font (size 1.27 1.27)) hide)
     )
@@
       (effects (font (size 1.27 1.27)) (justify right))
     )
-    (property "Footprint" "Resistor_SMD:R_1206_3216Metric" (at 65.278 224.79 90)
+    (property "Footprint" "Resistor_SMD:R_0805_2012Metric" (at 65.278 224.79 90)
       (effects (font (size 1.27 1.27)) hide)
     )
@@
   )
   (symbol (lib_id "Connector_Generic:Conn_01x03") (at 429.895 168.91 0) (unit 1)
-    (in_bom yes) (on_board yes) (dnp no) (fields_autoplaced)
+    (in_bom yes) (on_board yes) (dnp yes) (fields_autoplaced)
     (property "Reference" "J8" (at 433.07 168.275 0)
       (effects (font (size 1.27 1.27)) (justify left))
@@
       (effects (font (size 1.27 1.27)))
     )
-    (property "Footprint" "Resistor_SMD:R_1206_3216Metric" (at 61.722 201.93 90)
+    (property "Footprint" "Resistor_SMD:R_0805_2012Metric" (at 61.722 201.93 90)
       (effects (font (size 1.27 1.27)) hide)
     )
@@
       (effects (font (size 1.27 1.27)) (justify right))
     )
-    (property "Footprint" "Resistor_SMD:R_1206_3216Metric" (at 258.318 377.19 90)
+    (property "Footprint" "Resistor_SMD:R_0805_2012Metric" (at 258.318 377.19 90)
       (effects (font (size 1.27 1.27)) hide)
     )
@@
   )
   (symbol (lib_id "Switch:SW_DIP_x04") (at 242.57 308.61 0) (unit 1)
-    (in_bom yes) (on_board yes) (dnp no) (fields_autoplaced)
+    (in_bom yes) (on_board yes) (dnp yes) (fields_autoplaced)
     (property "Reference" "SW1" (at 242.57 297.18 0)
       (effects (font (size 1.27 1.27)))
@@
   )
   (symbol (lib_id "Connector_Generic:Conn_01x04") (at 488.315 78.74 0) (unit 1)
-    (in_bom yes) (on_board yes) (dnp no) (fields_autoplaced)
+    (in_bom yes) (on_board yes) (dnp yes) (fields_autoplaced)
     (property "Reference" "J4" (at 491.49 79.375 0)
       (effects (font (size 1.27 1.27)) (justify left))
@@
       (effects (font (size 1.27 1.27)) (justify right))
     )
-    (property "Footprint" "Resistor_SMD:R_1206_3216Metric" (at 258.318 316.23 90)
+    (property "Footprint" "Resistor_SMD:R_0805_2012Metric" (at 258.318 316.23 90)
       (effects (font (size 1.27 1.27)) hide)
     )
@@
   )
   (symbol (lib_id "MP4541GN-Z:MP4541GN-Z") (at 118.11 187.96 0) (mirror y) (unit 1)
-    (in_bom yes) (on_board yes) (dnp no) (fields_autoplaced)
+    (in_bom yes) (on_board yes) (dnp yes) (fields_autoplaced)
     (property "Reference" "B1" (at 102.87 181.61 0)
       (effects (font (size 1.27 1.27)))
@@
   )
   (symbol (lib_name "Conn_01x03_1") (lib_id "Connector_Generic:Conn_01x03") (at 161.29 139.7 0) (unit 1)
-    (in_bom yes) (on_board yes) (dnp no) (fields_autoplaced)
+    (in_bom yes) (on_board yes) (dnp yes) (fields_autoplaced)
     (property "Reference" "J3" (at 163.83 139.065 0)
       (effects (font (size 1.27 1.27)) (justify left))
@@
       (effects (font (size 1.27 1.27)))
     )
-    (property "Footprint" "Resistor_SMD:R_1206_3216Metric" (at 419.1 109.728 90)
+    (property "Footprint" "Resistor_SMD:R_0805_2012Metric" (at 419.1 109.728 90)
       (effects (font (size 1.27 1.27)) hide)
     )
@@
   )
   (symbol (lib_id "Switch:SW_DIP_x04") (at 242.57 340.36 0) (unit 1)
-    (in_bom yes) (on_board yes) (dnp no) (fields_autoplaced)
+    (in_bom yes) (on_board yes) (dnp yes) (fields_autoplaced)
     (property "Reference" "SW2" (at 242.57 328.93 0)
       (effects (font (size 1.27 1.27)))
@@
   )
   (symbol (lib_id "Connector_Generic:Conn_01x03") (at 429.895 133.35 0) (unit 1)
-    (in_bom yes) (on_board yes) (dnp no) (fields_autoplaced)
+    (in_bom yes) (on_board yes) (dnp yes) (fields_autoplaced)
     (property "Reference" "J5" (at 433.07 132.715 0)
       (effects (font (size 1.27 1.27)) (justify left))
@@
       (effects (font (size 1.27 1.27)) (justify left))
     )
-    (property "Footprint" "Capacitor_SMD:C_1206_3216Metric" (at 59.3852 215.9 0)
+    (property "Footprint" "Capacitor_SMD:C_0603_1608Metric" (at 59.3852 215.9 0)
       (effects (font (size 1.27 1.27)) hide)
     )
@@
       (effects (font (size 1.27 1.27)))
     )
-    (property "Footprint" "LED_SMD:LED_1206_3216Metric" (at 427.99 107.95 0)
+    (property "Footprint" "LED_SMD:LED_0603_1608Metric" (at 427.99 107.95 0)
       (effects (font (size 1.27 1.27)) hide)
     )
@@
       (effects (font (size 1.27 1.27)))
     )
-    (property "Footprint" "Resistor_SMD:R_1206_3216Metric" (at 223.52 339.598 90)
+    (property "Footprint" "Resistor_SMD:R_0805_2012Metric" (at 223.52 339.598 90)
       (effects (font (size 1.27 1.27)) hide)
     )
@@
       (effects (font (size 1.27 1.27)))
     )
-    (property "Footprint" "Resistor_SMD:R_1206_3216Metric" (at 217.17 310.388 90)
+    (property "Footprint" "Resistor_SMD:R_0805_2012Metric" (at 217.17 310.388 90)
       (effects (font (size 1.27 1.27)) hide)
     )
@@
       (effects (font (size 1.27 1.27) italic) (justify left))
     )
-    (property "Footprint" "Resistor_SMD:R_1206_3216Metric" (at 150.622 181.61 90)
+    (property "Footprint" "Resistor_SMD:R_0805_2012Metric" (at 150.622 181.61 90)
       (effects (font (size 1.27 1.27)) hide)
     )
@@
       (effects (font (size 1.27 1.27)))
     )
-    (property "Footprint" "Resistor_SMD:R_1206_3216Metric" (at 229.87 337.058 90)
+    (property "Footprint" "Resistor_SMD:R_0805_2012Metric" (at 229.87 337.058 90)
       (effects (font (size 1.27 1.27)) hide)
     )
@@
   )
   (symbol (lib_id "Connector_Generic:Conn_01x03") (at 429.895 145.415 0) (unit 1)
-    (in_bom yes) (on_board yes) (dnp no) (fields_autoplaced)
+    (in_bom yes) (on_board yes) (dnp yes) (fields_autoplaced)
     (property "Reference" "J6" (at 433.07 144.78 0)
       (effects (font (size 1.27 1.27)) (justify left))
@@
       (effects (font (size 1.27 1.27)))
     )
-    (property "Footprint" "Resistor_SMD:R_1206_3216Metric" (at 61.722 212.09 90)
+    (property "Footprint" "Resistor_SMD:R_0805_2012Metric" (at 61.722 212.09 90)
       (effects (font (size 1.27 1.27)) hide)
     )
@@
       (effects (font (size 1.27 1.27)))
     )
-    (property "Footprint" "Resistor_SMD:R_1206_3216Metric" (at 229.87 305.308 90)
+    (property "Footprint" "Resistor_SMD:R_0805_2012Metric" (at 229.87 305.308 90)
       (effects (font (size 1.27 1.27)) hide)
     )
@@
       (effects (font (size 1.27 1.27) italic) (justify left))
     )
-    (property "Footprint" "Resistor_SMD:R_1206_3216Metric" (at 121.412 106.68 90)
+    (property "Footprint" "Resistor_SMD:R_0805_2012Metric" (at 121.412 106.68 90)
       (effects (font (size 1.27 1.27)) hide)
     )
@@
       (effects (font (size 1.27 1.27) italic) (justify left))
     )
-    (property "Footprint" "Resistor_SMD:R_1206_3216Metric" (at 108.712 116.84 90)
+    (property "Footprint" "Resistor_SMD:R_0805_2012Metric" (at 108.712 116.84 90)
       (effects (font (size 1.27 1.27)) hide)
     )
@@
   )
   (symbol (lib_id "Connector_Generic:Conn_02x03_Odd_Even") (at 427.355 231.14 0) (unit 1)
-    (in_bom yes) (on_board yes) (dnp no) (fields_autoplaced)
+    (in_bom yes) (on_board yes) (dnp yes) (fields_autoplaced)
     (property "Reference" "J9" (at 428.625 223.52 0)
       (effects (font (size 1.27 1.27)))
@@
       (effects (font (size 1.27 1.27)) (justify right))
     )
-    (property "Footprint" "Resistor_SMD:R_1206_3216Metric" (at 154.178 193.04 90)
+    (property "Footprint" "Resistor_SMD:R_0805_2012Metric" (at 154.178 193.04 90)
       (effects (font (size 1.27 1.27)) hide)
     )
@@
   )
   (symbol (lib_id "Connector_Generic:Conn_01x03") (at 429.895 156.845 0) (unit 1)
-    (in_bom yes) (on_board yes) (dnp no) (fields_autoplaced)
+    (in_bom yes) (on_board yes) (dnp yes) (fields_autoplaced)
     (property "Reference" "J7" (at 433.07 156.21 0)
       (effects (font (size 1.27 1.27)) (justify left))
@@
       (effects (font (size 1.27 1.27)))
     )
-    (property "Footprint" "Resistor_SMD:R_1206_3216Metric" (at 223.52 307.848 90)
+    (property "Footprint" "Resistor_SMD:R_0805_2012Metric" (at 223.52 307.848 90)
       (effects (font (size 1.27 1.27)) hide)
     )
@@
       (effects (font (size 1.27 1.27)))
     )
-    (property "Footprint" "Resistor_SMD:R_1206_3216Metric" (at 92.71 46.482 90)
+    (property "Footprint" "Resistor_SMD:R_0805_2012Metric" (at 92.71 46.482 90)
       (effects (font (size 1.27 1.27)) hide)
     )
@@
       (effects (font (size 1.27 1.27)))
     )
-    (property "Footprint" "Resistor_SMD:R_1206_3216Metric" (at 210.82 312.928 90)
+    (property "Footprint" "Resistor_SMD:R_0805_2012Metric" (at 210.82 312.928 90)
       (effects (font (size 1.27 1.27)) hide)
     )
@@
   )
   (symbol (lib_id "Switch:SW_DIP_x01") (at 242.57 368.3 0) (unit 1)
-    (in_bom yes) (on_board yes) (dnp no) (fields_autoplaced)
+    (in_bom yes) (on_board yes) (dnp yes) (fields_autoplaced)
     (property "Reference" "SW3" (at 242.57 361.95 0)
       (effects (font (size 1.27 1.27)))
@@
       (effects (font (size 1.27 1.27)) (justify right))
     )
-    (property "Footprint" "Resistor_SMD:R_1206_3216Metric" (at 128.778 201.93 90)
+    (property "Footprint" "Resistor_SMD:R_0805_2012Metric" (at 128.778 201.93 90)
       (effects (font (size 1.27 1.27)) hide)
     )
@@
       (effects (font (size 1.27 1.27)) (justify right))
     )
-    (property "Footprint" "Resistor_SMD:R_1206_3216Metric" (at 258.318 351.79 90)
+    (property "Footprint" "Resistor_SMD:R_0805_2012Metric" (at 258.318 351.79 90)
       (effects (font (size 1.27 1.27)) hide)
     )
@@
       (effects (font (size 1.27 1.27)))
     )
-    (property "Footprint" "Resistor_SMD:R_1206_3216Metric" (at 210.82 344.678 90)
-      (effects (font (size 1.27 1.27)) hide)
-    )
+    (property "Footprint" "Resistor_SMD:R_0805_2012Metric" (at 210.82 344.678 90)
+      (effects (font (size 1.27 1.27)) hide)
+    )
